File: multiplier/multiplier.kicad_sch (KiCad schematic)
At the start: 6 parts, among them J1 Screw_Terminal_01x01, J2 Screw_Terminal_01x01, J3 Screw_Terminal_01x08, U1 AD633ARZ-R7, U2 AD633ARZ-R7

Commit message: Update
Changed lines of the file:
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@@
 	(wire
 		(pts
-			(xy 158.75 105.41) (xy 154.94 105.41)
+			(xy 154.94 118.11) (xy 220.98 118.11)
 		)
 		(stroke
@@
 	(wire
 		(pts
-			(xy 175.26 97.79) (xy 180.34 97.79)
+			(xy 171.45 97.79) (xy 180.34 97.79)
 		)
 		(stroke
@@
 	(wire
 		(pts
-			(xy 158.75 109.22) (xy 158.75 105.41)
-		)
-		(stroke
-			(width 0)
-			(type default)
-		)
-	)
-	(wire
-		(pts
 			(xy 59.69 162.56) (xy 38.1 162.56)
 		)
@@
 	(wire
 		(pts
-			(xy 59.69 100.33) (xy 73.66 100.33)
+			(xy 59.69 109.22) (xy 73.66 109.22)
 		)
 		(stroke
@@
 	(wire
 		(pts
-			(xy 220.98 109.22) (xy 158.75 109.22)
-		)
-		(stroke
-			(width 0)
-			(type default)
-		)
-	)
-	(wire
-		(pts
-			(xy 220.98 100.33) (xy 220.98 109.22)
+			(xy 220.98 100.33) (xy 220.98 118.11)
 		)
 		(stroke
@@
 	(wire
 		(pts
-			(xy 119.38 104.14) (xy 129.54 104.14)
-		)
-		(stroke
-			(width 0)
-			(type default)
-		)
-	)
-	(wire
-		(pts
-			(xy 105.41 86.36) (xy 105.41 90.17)
+			(xy 119.38 113.03) (xy 129.54 113.03)
+		)
+		(stroke
+			(width 0)
+			(type default)
+		)
+	)
+	(wire
+		(pts
+			(xy 105.41 95.25) (xy 105.41 99.06)
 		)
 		(stroke
@@
 	)
 	(label "V3"
-		(at 105.41 86.36 0)
+		(at 105.41 95.25 0)
 		(effects
 			(font
@@
 	)
 	(label "Control_in"
-		(at 59.69 100.33 0)
+		(at 59.69 109.22 0)
 		(effects
 			(font
@@
 	(global_label "V2"
 		(shape input)
-		(at 175.26 97.79 180)
+		(at 171.45 97.79 180)
 		(fields_autoplaced yes)
 		(effects
@@
 		)
 		(property "Intersheetrefs" "${INTERSHEET_REFS}"
-			(at 169.9767 97.79 0)
+			(at 166.1667 97.79 0)
 			(effects
 				(font
@@
 	)
 	(sheet
-		(at 73.66 90.17)
+		(at 73.66 99.06)
 		(size 45.72 27.94)
 		(exclude_from_sim no)
@@
 		)
 		(property "Sheetname" "Amplifiers"
-			(at 73.66 89.4584 0)
+			(at 73.66 98.3484 0)
 			(effects
 				(font
@@
 		)
 		(property "Sheetfile" "amplifiers.kicad_sch"
-			(at 73.66 118.6946 0)
+			(at 73.66 127.5846 0)
 			(effects
 				(font
@@
 		)
 		(pin "Command_out" input
-			(at 73.66 100.33 180)
+			(at 73.66 109.22 180)
 			(effects
 				(font
@@
 		)
 		(pin "Twin_in" input
-			(at 119.38 104.14 0)
+			(at 119.38 113.03 0)
 			(effects
 				(font
@@
 		)
 		(pin "V3" input
-			(at 105.41 90.17 90)
+			(at 105.41 99.06 90)
 			(effects
 				(font
@@
 	)
 	(sheet
-		(at 129.54 93.98)
+		(at 129.54 102.87)
 		(size 25.4 20.32)
 		(exclude_from_sim no)
@@
 		)
 		(property "Sheetname" "Twin T"
-			(at 129.54 93.2684 0)
+			(at 129.54 102.1584 0)
 			(effects
 				(font
@@
 		)
 		(property "Sheetfile" "twin_t.kicad_sch"
-			(at 129.54 114.8846 0)
+			(at 129.54 123.7746 0)
 			(effects
 				(font
@@
 		)
 		(pin "Analog_in" input
-			(at 154.94 105.41 0)
+			(at 154.94 118.11 0)
 			(effects
 				(font
@@
 		)
 		(pin "Twin_out" input
-			(at 129.54 104.14 180)
-			(effects
-				(font
+			(at 129.54 113.03 180)
+			(effects
+				(font
