File: multiplier/twin_t.kicad_sch (KiCad schematic)
At the start: 13 parts, among them U7 LT1793AIS8-PBF, U8 LT1793AIS8-PBF, U9 LT1793AIS8-PBF

Commit message: Update
Parts:
- removed R14, R15: R, symbol Device:R
Connections:
- net Twin_out: now also U9.2 (-INA)
