File: current_measure_board/current_measure_board.kicad_sch (KiCad schematic)
At the start: 22 parts, among them U1 LT6370HMS8-TRPBF, U2 LT1793AIS8-PBF, U3 LT1793AIS8-PBF, U4 LT1793AIS8-PBF

Commit message: old 250H checkpoint 1 code preserved here
Parts:
- added R2: TS63Y201KR10, Custom_trimpot:TRIM_TS63Y201KR10, symbol Custom_Potentiometers:TS63Y201KR10
- C1, C2: footprint (none) -> Custom_capacitors:CAPC2012X140N(50pF 1206 1 C0G 100V)
- C3, C4, C5: footprint (none) -> Custom_capacitors:CAPC2012X145N(200pF 0805 0.1err)
- R1: footprint (none) -> Custom_resistors:RES_TNPW0603_VIS-L(2.7k Ohm 0603 0.1err)
- R3: value 1k -> 4.2k; footprint (none) -> Custom_resistors:RESC2012X55N(4.02k Ohm 0805 0.1err)
- R4, R7: value 4k -> 4.2k; footprint (none) -> Custom_resistors:RESC2012X55N(4.02k Ohm 0805 0.1err)
- R6: value 1k -> 3.92k; footprint (none) -> Custom_resistors:RES_TNPW0805_VIS-L(3.92k Ohm 0805 0.1)
- R8, R9: footprint (none) -> Custom_resistors:RESC2012X55N(500 Ohm 0805 0.05err)
- TP1, TP2, TP3, TP4, TP5, TP6: footprint (none) -> Custom_trimpot:PAD_EXT_2.54x5.08mm
- U1: footprint 05-08-1660_ADI -> Custom_amplifiers:LT6370HMS8_TRPBF_L
- U2, U3, U4: footprint SO-8_S_LIT -> Custom_amplifiers:LT1793AIS_8_PBF
Connections:
- net GND: now also R2.2; no longer R6.2
- net Vminus: no longer U1.4 (V-), U2.4 (V-), U3.4 (V-), U4.4 (V-)
- net Vplus: no longer U1.7 (V+), U2.7 (V+), U3.7 (V+), U4.7 (V+)
- new net: R2.1, R6.2
- new net power_buffer_minus/terminal_side: U3.4 (V-)
- new net power_buffer_minus1/terminal_side: U1.4 (V-)
- new net power_buffer_minus2/terminal_side: U2.4 (V-)
- new net power_buffer_minus3/terminal_side: U4.4 (V-)
- new net power_buffer_plus/terminal_side: U3.7 (V+)
- new net power_buffer_plus1/terminal_side: U1.7 (V+)
- new net power_buffer_plus2/terminal_side: U2.7 (V+)
- new net power_buffer_plus3/terminal_side: U4.7 (V+)
- no-connect marks 9 -> 10
Other:
- added sheet power_buffer_minus (power_buffer_minus.kicad_sch)
- added sheet power_buffer_minus1 (power_buffer_minus.kicad_sch)
- added sheet power_buffer_minus2 (power_buffer_minus.kicad_sch)
- added sheet power_buffer_minus3 (power_buffer_minus.kicad_sch)
- added sheet power_buffer_plus (power_buffer_plus.kicad_sch)
- added sheet power_buffer_plus1 (power_buffer_plus.kicad_sch)
- added sheet power_buffer_plus2 (power_buffer_plus.kicad_sch)
- added sheet power_buffer_plus3 (power_buffer_plus.kicad_sch)
- moved on the sheet: R6

Commit message: high impedance section draft done
Parts:
- TP4, TP5: footprint Custom_trimpot:PAD_EXT_2.54x5.08mm -> Custom_testpoint:PAD_EXT_0.635x2.54mm
Changed lines of the file:
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@@
 			)
 		)
-		(property "Footprint" "Custom_trimpot:PAD_EXT_2.54x5.08mm"
+		(property "Footprint" "Custom_testpoint:PAD_EXT_0.635x2.54mm"
 			(at 33.02 171.45 0)
 			(effects
@@
 			)
 		)
-		(property "Footprint" "Custom_trimpot:PAD_EXT_2.54x5.08mm"
+		(property "Footprint" "Custom_testpoint:PAD_EXT_0.635x2.54mm"
 			(at 33.02 162.56 0)
 			(effects

Commit message: current board update
Parts:
- added C26: 50p, Custom_capacitors:CAPC2012X140N(50pF 1206 1 C0G 100V), symbol Device:C
- added R10: 4.02k, Custom_resistors:RESC2012X55N(4.02k Ohm 0805 0.1err), symbol Device:R
- added TP10: TestPoint, Custom_testpoint:PAD_EXT_0.635x2.54mm, symbol Connector:TestPoint
- added TP7, TP8, TP9: TestPoint, Custom_trimpot:PAD_EXT_2.54x5.08mm, symbol Connector:TestPoint
- added U5: LT1793AIS8-PBF, Custom_amplifiers:LT1793AIS_8_PBF, symbol Custom_amplifier:LT1793AIS8-PBF
- R3, R4, R7: value 4.2k -> 4.02k
Connections:
- net GND: now also TP7.1, TP9.1, U5.3 (+INA)
- new net Current_in: C26.2, R10.2, TP10.1, U5.2 (-INA)
- new net Current_meas: C26.1, R10.1, TP8.1, U5.6 (OUT)
- new net power_buffer_minus4/terminal_side: U5.4 (V-)
- new net power_buffer_plus4/terminal_side: U5.7 (V+)
- no-connect marks 10 -> 13
Other:
- added sheet power_buffer_minus4 (power_buffer_minus.kicad_sch)
- added sheet power_buffer_plus4 (power_buffer_plus.kicad_sch)
